File: STTS22H_Temperature_Sensor.kicad_pcb (KiCad board)
At the start: 2 copper layers, 30.2 x 30.2 mm, 15 parts, among them J1 JST_SH_SM06B-SRSS-TB_1x06-1MP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, J4 Conn_01x04, U1 M24C02-FMN, U2 STTS22HTR

Commit message: Change to 10K pullup resistor on interrupt line.
Parts:
- R1: value 100K -> 10K
Changed lines of the file:
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@@
 			)
 		)
-		(property "Value" "100K"
+		(property "Value" "10K"
 			(at 0 1.43 90)
 			(layer "F.Fab")
@@
 			)
 		)
-		(property "MPN" ""
+		(property "MPN" "C25804"
 			(at 0 0 270)
 			(unlocked yes)
@@
 			)
 		)
-		(property "Feeder" ""
+		(property "Feeder" "8mm"
 			(at 0 0 270)
 			(unlocked yes)
@@
 		(start 40.249999 48.0222)
 		(end 41.9003 48.0222)
-		(width 0.6)
+		(width 0.3)
 		(layer "F.Cu")
 		(net 1)
@@
 		(start 39.6 46.1728)
 		(end 41.9003 46.1728)
-		(width 0.6)
+		(width 0.3)
 		(layer "F.Cu")
 		(net 2)
@@
 	)
 	(segment
+		(start 48.05 48.0125)
+		(end 47.177954 48.884546)
+		(width 0.3)
+		(layer "F.Cu")
+		(net 3)
+	)
+	(segment
+		(start 60.1 45.35)
+		(end 60.35 45.6)
+		(width 0.3)
+		(layer "F.Cu")
+		(net 3)
+	)
+	(segment
+		(start 60.1 44.5)
+		(end 60.1 45.35)
+		(width 0.3)
+		(layer "F.Cu")
+		(net 3)
+	)
+	(segment
+		(start 59.15 43.55)
+		(end 60.1 44.5)
+		(width 0.3)
+		(layer "F.Cu")
+		(net 3)
+	)
+	(segment
 		(start 39.6 48.669092)
 		(end 39.6 48.0222)
@@
 	)
 	(segment
-		(start 48.05 48.0125)
-		(end 47.177954 48.884546)
+		(start 39.815454 48.884546)
+		(end 39.6 48.669092)
+		(width 0.3)
+		(layer "F.Cu")
+		(net 3)
+	)
+	(segment
+		(start 60.35 45.6)
+		(end 61.409284 45.6)
 		(width 0.3)
 		(layer "F.Cu")
@@
 		(width 0.3)
 		(layer "F.Cu")
-		(net 3)
-	)
-	(segment
-		(start 60.1 45.35)
-		(end 60.35 45.6)
-		(width 0.3)
-		(layer "F.Cu")
-		(net 3)
-	)
-	(segment
-		(start 60.1 44.5)
-		(end 60.1 45.35)
-		(width 0.3)
-		(layer "F.Cu")
-		(net 3)
-	)
-	(segment
-		(start 59.15 43.55)
-		(end 60.1 44.5)
-		(width 0.3)
-		(layer "F.Cu")
-		(net 3)
-	)
-	(segment
-		(start 60.35 45.6)
-		(end 61.409284 45.6)
-		(width 0.3)
-		(layer "F.Cu")
-		(net 3)
-	)
-	(segment
-		(start 39.815454 48.884546)
-		(end 39.6 48.669092)
-		(width 0.3)
-		(layer "F.Cu")
