File: STTS22H_Temperature_Sensor.kicad_sch (KiCad schematic)
At the start: 9 parts, among them J1 JST_SH_SM06B-SRSS-TB_1x06-1MP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, J4 Conn_01x04, U1 M24C02-FMN, U2 STTS22HTR

Commit message: Change to 10K pullup resistor on interrupt line.
Parts:
- R1: value 100K -> 10K; Feeder (none) -> 8mm; MPN (none) -> C25804
Changed lines of the file:
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@@
 			)
 		)
-		(property "Value" "100K"
+		(property "Value" "10K"
 			(at 100.33 30.4799 0)
 			(effects
@@
 			)
 		)
-		(property "MPN" ""
+		(property "MPN" "C25804"
 			(at 97.79 29.21 0)
 			(effects
@@
 			)
 		)
-		(property "Feeder" ""
+		(property "Feeder" "8mm"
 			(at 97.79 29.21 0)
 			(effects
